File: MatterRGB.kicad_sch (KiCad schematic)
At the start: 49 parts, among them J1 USB4105, J2 S4B-PH-K-S, J4 S2B-XH-A-1, J5 S2B-PH-K-S, SW1 NO, SW2 NO, U1 FUSB302B01MPX, U2 ESP32-S3-WROOM-1-N8R8, U3 DRV8955, U5 LMR50410Y3FQDBVRQ1

Commit message: Lots of other stuff
Other:
- note added: "change to 3v3"
Changed lines of the file:
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@@
 	(generator_version "9.0")
 	(paper "A4")
+	(circle
+		(center 165.1 97.79)
+		(radius 4.836)
+		(stroke
+			(width 0)
+			(type default)
+		)
+		(fill
+			(type none)
+		)
+	)
+	(text "change to 3v3"
+		(exclude_from_sim no)
+		(at 165.862 91.44 0)
+		(effects
+			(font
+				(size 1.27 1.27)
+			)
+		)
+	)
 	(junction
 		(at 60.96 64.77)

Commit message: Added new connector/mounting strategy
Parts:
- removed J1: USB4105, Connector_USB:USB_C_Receptacle_GCT_USB4105-xx-A_16P_TopMnt_Horizontal, symbol partywagon112_partdb:USB4105-GF-A
- removed J2: S4B-PH-K-S, Connector_JST:JST_PH_S4B-PH-K_1x04_P2.00mm_Horizontal, symbol partywagon112_partdb:S4B-PH-K-S
- removed J4: S2B-XH-A-1, Connector_JST:JST_XH_S2B-XH-A-1_1x02_P2.50mm_Horizontal, symbol partywagon112_partdb:S2B-XH-A-1
- removed J5: S2B-PH-K-S, Connector_JST:JST_PH_S2B-PH-K_1x02_P2.00mm_Horizontal, symbol partywagon112_partdb:S2B-PH-K-S
- removed U2: ESP32-S3-WROOM-1-N8R8, RF_Module:ESP32-S3-WROOM-1, symbol partywagon112_partdb:ESP32-S3-WROOM-1-N8R8
- removed U5: LMR50410Y3FQDBVRQ1, Package_TO_SOT_SMD:SOT-23-6, symbol partywagon112_fred_partdb:LMR50410Y3FQDBVRQ1
- added C18: 100n, Capacitor_SMD:C_0402_1005Metric, symbol partywagon112_fred_partdb:GCM155R71H104KE02J
- added D4: RCLAMP0582B.TCT, Package_TO_SOT_SMD:SOT-416, symbol partywagon112_partdb:RCLAMP0582B.TCT
- added J1: CDM806-04A-MP-F011-67, PCM_PartyWagon112_Connector_M8:CUI_CDM806-04A-MP-F011-67, symbol partywagon112_partdb:CDM806-04A-MP-F011-67
- added J2: USB4115-03-C, Connector_USB:USB_C_Receptacle_GCT_USB4115-03-C, symbol partywagon112_partdb:USB4115-03-C
- added J5: CDM802-08A-FP-F010-67, PCM_PartyWagon112_Connector_M8:CUI_CDM802-08A-FP-F010-67, symbol partywagon112_partdb:CDM802-08A-FP-F010-67
- added R12, R13: 10k, Resistor_SMD:R_0402_1005Metric, symbol partywagon112_partdb:CR0402AFX-1002GAS
- added R14, R15: 0, Resistor_SMD:R_0402_1005Metric, symbol partywagon112_partdb:CR0402AJ/-000GLF
- added U2: ESP32-S3-WROOM-1U-N8R8, RF_Module:ESP32-S3-WROOM-1U, symbol partywagon112_partdb:ESP32-S3-WROOM-1U-N8R8
- added U5: LMR51610YFDBVR, Package_TO_SOT_SMD:SOT-23-6, symbol partywagon112_partdb:LMR51610YFDBVR
Connections:
- net +3V3: now also R1.1, R13.1, U2.2 (3V3), U5.3 (FB)
- net 3V3_SW: now also U5.6 (SW)
- net BOOT: now also U2.27 (IO0)
- net CC1: now also D4.1 (K1), J2.A5 (CC1), R14.2
- net CC2: now also D4.2 (K2), J2.B5 (CC2), R15.2
- net GND: now also C18.2, D4.3 (A), J1.2 (Pin_2), J2.A1 (GND), J2.A12 (GND), J2.B1 (GND), J2.B12 (GND), J2.S1 (SHIELD), J5.3 (Pin_3), J5.4 (Pin_4), U2.1 (GND), U2.40 (GND), U2.41 (GND), U5.2 (GND)
- net IN0: now also C8.1, R5.2, R6.1, J5.1 (Pin_1), U2.10 (IO17); no longer R6.2
- net IN1: now also C18.1, J5.2 (Pin_2), R12.1, R13.2, U2.11 (IO18); no longer U3.20 (IN1)
- net INT_N: now also U2.19 (IO11)
- net MODE: now also U2.25 (IO48)
- net OUT1: now also J5.5 (Pin_5)
- net OUT2: now also J5.6 (Pin_6)
- net OUT3: now also J5.7 (Pin_7)
- net OUT4: now also J5.8 (Pin_8)
- net RESET: now also U2.3 (EN)
- net RSVD/EN1: now also U2.32 (IO39)
- net SCL: now also U2.17 (IO9)
- net SDA: now also U2.12 (IO8)
- net TOFF/EN2: now also U2.33 (IO40)
- net USB_D+: now also J2.A6 (D+), J2.B6 (D+), U2.14 (USB_D+)
- net USB_D-: now also J2.A7 (D-), J2.B7 (D-), U2.13 (USB_D-)
- net VBUS: now also J2.A4 (VBUS), J2.A9 (VBUS), J2.B4 (VBUS), J2.B9 (VBUS)
- net VDC: now also U5.4 (EN), U5.5 (VIN)
- net VDD: no longer R1.1
- net VREF12/EN3: now also U2.34 (IO41)
- net VREF12/EN4: now also U2.35 (IO42)
- net ~{FAULT}: now also U2.38 (IO2)
- net ~{SLEEP}: now also U2.18 (IO10)
- net at LED2.2 (A): now also U2.8 (IO15)
- net at F1.2: now also J1.1 (Pin_1)
- net at C28.1: now also U5.1 (CB)
- net IN2 renamed OUT2_CPU
- net OUT2_CPU: now also U2.21 (IO13)
- net IN3 renamed OUT3_CPU
- net OUT3_CPU: now also U2.23 (IO21)
- net IN4 renamed OUT4_CPU
- net OUT4_CPU: now also U2.24 (IO47)
- new net: J1.3 (Pin_3), R15.1
- new net: J1.4 (Pin_4), R14.1
- new net IN0_MCU: R6.2
- new net IN1_MCU: R12.2
- new net OUT1_CPU: U2.20 (IO12), U3.20 (IN1)
Other:
- note removed: "change to 3v3"
- moved on the sheet: C1, C10, C11, C12, C13, C14, C15, C16, C17, C2, C28, C29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
