File: hardware/inputs.kicad_sch (KiCad schematic)
At the start: 13 parts, among them Q1 2N7002KL3A-TP, U4 ADA4098-2BCPZ-RL7, U6 TPS7B4255DBVR

Commit message: Finished draft layout of muCM update.
Parts:
- removed C18, C8: 10 nF, Resistor_SMD:R_0603_1608Metric, symbol partywagon112_partdb:GCM188R71H103KA37D
- removed C20: 1u, Capacitor_SMD:C_0603_1608Metric, symbol partywagon112_partdb:GRT188R61H105KE13D
- removed C21: 100n, Capacitor_SMD:C_0805_2012Metric, symbol partywagon112_partdb:KAS21KR72A104KU
- removed Q1: 2N7002KL3A-TP, Package_DFN_QFN:Diodes_DFN1006-3, symbol partywagon112_partdb:2N7002KL3A-TP
- removed R12, R5: 2.2kR, Resistor_SMD:R_0603_1608Metric, symbol partywagon112_partdb:CMP0603QFX-2201ELF
- removed R14: 10k, Resistor_SMD:R_0402_1005Metric, symbol partywagon112_partdb:CR0402AFX-1002GAS
- removed U6: TPS7B4255DBVR, Package_TO_SOT_SMD:SOT-23-5, symbol partywagon112_partdb:TPS7B4255DBVR
- added C18, C8: 10nF, Capacitor_SMD:C_0603_1608Metric, symbol partywagon112_partdb:CL10B103KC8WPNC
- added R12, R5: 10k, Resistor_SMD:R_0402_1005Metric, symbol partywagon112_partdb:CR0402AFX-1002GAS
Connections:
- net GND: now also C18.2, C8.2
- net IN0: now also U4.3 (+), C8.1, R12.2; no longer U4.7 (+)
- net IN0_MCU: now also U4.1, U4.2 (-); no longer U4.8 (-), U4.9
- net IN1: now also U4.7 (+), C18.1, R5.2; no longer U4.3 (+)
- net IN1_MCU: now also U4.8 (-), U4.9; no longer U4.1, U4.2 (-)
- new net +3.3VP: R12.1, R5.1
